File: electrical schematics/Power Distribution PCB Schematic/Power Distribution PCB Schematic.kicad_sch (KiCad schematic)
At the start: 0 parts

Commit message: Reorganizing
Mostly electrical file stuff
Parts:
- added 10k1, 1k1, 33k1, 470ohm1, 470ohm2, R1: R_US, symbol Device:R_US
- added 330uF1: C, symbol Device:C
- added 5V_Converter1: ~, symbol Rover_Project:5V_Voltage_Regulator_-_D36V28F5
- added A1: RaspberryPi_Pico, Module:RaspberryPi_Pico_Common_Unspecified, symbol MCU_Module:RaspberryPi_Pico
- added C1, C10, C3, C7: 220uF, symbol Device:C_Polarized
- added C2, C4, C6, C9: 68nF, symbol Device:C
- added C5, C8: 10uF, symbol Device:C
- added D1, D2, D3, D4: LED, symbol Device:LED
- added F1: Fuse, symbol Device:Fuse
- added GPS_Module1: ~, symbol Rover_Project:GPS_Module
- added J1: XT60_Port, symbol Connector_Generic:Conn_01x02
- added J10, J11, J12, J9: Encoder_Header, symbol Connector_Generic:Conn_01x03
- added J13: 6VA_Converter_Input_Screw, symbol Connector:Screw_Terminal_01x02
- added J14: 6VB_Converter_Input_Screw, symbol Connector:Screw_Terminal_01x02
- added J15: 6VA_Converter_Output_Screw, symbol Connector:Screw_Terminal_01x02
- added J16: 6VA_Servo_Power_Screw, symbol Connector:Screw_Terminal_01x02
- added J17: 6VB_Servo_Power_Screw, symbol Connector:Screw_Terminal_01x02
- added J18: 6VB_Converter_Output_Screw, symbol Connector:Screw_Terminal_01x02
- added J19: ServoPWM_Header, symbol Connector_Generic:Conn_01x05
- added J2: On/Off_Switch_Screw_Terminal, symbol Connector:Screw_Terminal_01x02
- added J3: IMU_Header, symbol Connector_Generic:Conn_01x05
- added J4: Raspberry_Pi_4, symbol Connector:Raspberry_Pi_4
- added J5, J6, J7, J8: BDC_Motor_Screw_Terminal, symbol Connector:Screw_Terminal_01x03
- added R10, R11, R12, R13, R14, R15, R16, R17: 1k, symbol Device:R_US
- added R2, R3, R4, R5, R6, R7, R8, R9: 2k, symbol Device:R_US
- added U1: BDC_DRIVER_1, Package_SO:SSOP-24_5.3x8.2mm_P0.65mm, symbol Driver_Motor:TB6612FNG
- added U2: BDC_DRIVER_2, Package_SO:SSOP-24_5.3x8.2mm_P0.65mm, symbol Driver_Motor:TB6612FNG
Connections:
- new net: J4.13 (GPIO27/SDIO_DAT3), R13.1, R7.1
- new net: J11.2 (C2), R13.2
- new net: 1k1.2, D1.2 (A)
- new net: J5.1 (M+), U1.1 (AO1), U1.2 (AO1)
- new net: J6.1 (M+), U1.11 (BO1), U1.12 (BO1)
- new net: A1.6 (GPIO4), U1.15 (PWMB)
- new net: A1.1 (GPIO0), U1.16 (BIN2)
- new net: A1.2 (GPIO1), U1.17 (BIN1)
- new net: A1.9 (GPIO6), U1.19 (STBY)
- new net: A1.5 (GPIO3), U1.21 (AIN1)
- new net: A1.4 (GPIO2), U1.22 (AIN2)
- new net: A1.7 (GPIO5), U1.23 (PWMA)
- new net: J5.2 (M-), U1.5 (AO2), U1.6 (AO2)
- new net: J6.2 (M-), U1.7 (BO2), U1.8 (BO2)
- new net: 470ohm2.1, C10.1, C8.1, C9.1, J17.1 (Pin_1), J18.1 (Pin_1)
- new net: D2.2 (A), R1.2
- new net: 10k1.1, 33k1.1, A1.31 (GPIO26_ADC0)
- new net: A1.10 (GPIO7), U2.16 (BIN2)
- new net: A1.11 (GPIO8), U2.17 (BIN1)
- new net: A1.12 (GPIO9), U2.22 (AIN2)
- new net: A1.14 (GPIO10), U2.21 (AIN1)
- new net: A1.15 (GPIO11), U2.15 (PWMB)
- new net: A1.16 (GPIO12), U2.23 (PWMA)
- new net: A1.17 (GPIO13), U2.19 (STBY)
- new net: A1.27 (GPIO21), J4.8 (GPIO14/UART_TXD)
- new net: A1.29 (GPIO22), J4.10 (GPIO15/UART_RXD)
- new net: A1.35 (ADC_VREF), A1.37 (3V3_EN)
- new net: J4.1 (3V3), J4.17 (3V3)
- new net: J19.2 (Pin_2), J4.11 (GPIO17/SPI1_~{CE1})
- new net: J19.3 (Pin_3), J4.12 (GPIO18/SPI1_~{CE0}/PCM_CLK/PWM0)
- new net: J4.15 (GPIO22/SDIO_CLK), R14.1, R2.1
- new net: J4.16 (GPIO23/SDIO_CMD), R15.1, R3.1
- new net: J4.18 (GPIO24/SDIO_DAT0), R10.1, R4.1
- new net: GPS_Module1.1 (PPS), J4.21 (MISO_SPI0/GPIO09)
- new net: J4.22 (GPIO25/SDIO_DAT1), R11.1, R5.1
- new net: GPS_Module1.2 (RXD), J4.24 (~{CE0}_SPI0/GPIO08)
- new net: GPS_Module1.3 (TXD), J4.26 (~{CE1}_SPI0/GPIO07)
- new net: J4.29 (GPCLK1/GPIO05), R17.1, R9.1
- new net: J3.4 (SDA), J4.3 (SDA_I2C1/GPIO02)
- new net: J4.31 (GPCLK2/GPIO06), R16.1, R8.1
- new net: J19.4 (Pin_4), J4.35 (GPIO19/SPI1_MISO/PCM_FS)
- new net: J19.1 (Pin_1), J4.36 (GPIO16/SPI1_~{CE2})
- new net: J4.37 (GPIO26/SDIO_DAT2), R12.1, R6.1
- new net: J19.5 (Pin_5), J4.38 (GPIO20/SPI1_MOSI/PCM_DIN/PWM1)
- new net: J3.3 (SCL), J4.5 (SCL_I2C1/GPIO03)
- new net: J3.5 (INT), J4.7 (GPCLK0/GPIO04)
- new net: 470ohm2.2, D4.2 (A)
- new net: J9.1 (C1), R14.2
- new net: 470ohm1.2, D3.2 (A)
- new net: J11.1 (C1), R12.2
- new net: 5V_Converter1.1 (Vout), F1.2
- new net: J7.1 (M+), U2.1 (AO1), U2.2 (AO1)
- new net: J8.1 (M+), U2.11 (BO1), U2.12 (BO1)
- new net: J7.2 (M-), U2.5 (AO2), U2.6 (AO2)
- new net: J8.2 (M-), U2.7 (BO2), U2.8 (BO2)
- new net: J12.1 (C1), R16.2
- new net: 470ohm1.1, C3.1, C4.1, C5.1, J15.1 (Pin_1), J16.1 (Pin_1)
- new net: J12.2 (C2), R17.2
- new net: J9.2 (C2), R15.2
- new net: J10.1 (C1), R10.2
- new net: J10.2 (C2), R11.2
- new net 12V_Bus: 1k1.1, 330uF1.1, 33k1.2, 5V_Converter1.4 (Vin), C6.1, C7.1, J1.1 (12V_raw), J13.1 (Pin_1), J14.1 (Pin_1), J2.1 (Pin_1), J2.2 (Pin_2), U1.24 (VM1), U2.24 (VM1)
- new net 5V_Bus: A1.39 (VSYS), C1.1, C2.1, F1.1, GPS_Module1.5 (VCC), J10.3 (VCC), J11.3 (VCC), J12.3 (VCC), J3.1 (VCC), J4.2 (5V), J4.4 (5V), J9.3 (VCC), R1.1, U1.20 (VCC), U2.20 (VCC)
- new net GND: 10k1.2, 330uF1.2, 5V_Converter1.2 (GND), A1.13 (GND), A1.18 (GND), A1.23 (GND), A1.28 (GND), A1.3 (GND), A1.38 (GND), A1.8 (GND), C1.2, C10.2, C2.2, C3.2, C4.2, C5.2, C6.2, C7.2, C8.2, C9.2, D1.1 (K), D2.1 (K), D3.1 (K), D4.1 (K), GPS_Module1.4 (GND), J1.2 (GND), J13.2 (Pin_2), J14.2 (Pin_2), J15.2 (Pin_2), J16.2 (Pin_2), J17.2 (Pin_2), J18.2 (Pin_2), J3.2 (GND), J4.14 (GND), J4.20 (GND), J4.25 (GND), J4.30 (GND), J4.34 (GND), J4.39 (GND), J4.6 (GND), J4.9 (GND), J5.3 (GND), J6.3 (GND), J7.3 (GND), J8.3 (GND), R2.2, R3.2, R4.2, R5.2, R6.2, R7.2, R8.2, R9.2, U1.10 (PGND2), U1.18 (GND), U1.3 (PGND1), U1.4 (PGND1), U1.9 (PGND2), U2.10 (PGND2), U2.18 (GND), U2.3 (PGND1), U2.4 (PGND1), U2.9 (PGND2)
- no-connect marks 0 -> 25
Other:
- note added: "C1"
- note added: "C2"
- note added: "Comes with internal pull-up resistors for I2C communication"
- note added: "Converting 5V outputs to 3.3V for Pico using voltage dividers"
- note added: "Double check that all signal lines output 3.3V highs NOT 5V = damage"
- note added: "GND"
- note added: "Had to add this short to represent the external switch as connected for the ERC to work."
- note added: "INT"
- note added: "M+"
- note added: "M-"
- note added: "Must first disable SPI to use UART communication on GPIO07 & GPIO08 pins"
- note added: "Not sure why I didn't do this in first place but I can feed both converters with the same 12V filtered wire, no need for seperate inputs"
- note added: "SCL"
- note added: "SDA"
- note added: "VCC"
- note added: "VCC pins provide 5V for powering encoders, not the motors. Need screw terminals for M- and M+ lines only, regular GPIO headers for encoder wires"
- note added: "Voltage divider output for battery voltage monitoring"
- note added: "supplies 3.3V to the ADC reference pin"
